File: Lysergic25.kicad_pcb (KiCad board)
At the start: 2 copper layers, 99.1 x 99.1 mm, 111 parts, among them J1 Breakout, Q1 Q_NPN_BCE, SW1 SW_PUSH, U1 Pro_Micro, U2 PRTR5V0U2X

Commit message: _
Parts:
- Trrs2: moved to F.Cu
- moved Trrs1 2.95 mm to (66.5, 83.8)
- moved Trrs2 2.77 mm to (9.63, 83.9), turned to 0 degrees
Routing:
- net SDA: track 147.5 -> 134.2 mm, vias 3 -> 2
- net GND: track 42.2 -> 38.2 mm, vias 151 -> 153
- net SCL: track 131.3 -> 135.2 mm
- net ROW0: track 226.5 -> 228.0 mm, vias 3 -> 2
- net VCC: track 796.1 -> 794.9 mm, vias 22 -> 24
- net Net-(MX4-Pad4): vias 0 -> 1
Other:
- board text added: "JLCJLCJLCJLC"
- board text added: "REV 1"
